Commit message: assme symmetric dual hand at initialization & tune the parameter

File: src/curobo/content/assets/robot/shadow_hand/right_sim.urdf (robot description, URDF)
Before this commit: robot right_shadow_hand, 25 links, 24 joints
Links:
- removed link rh_forearm
- removed link rh_wrist
Joints:
- removed joint rh_WRJ1
- removed joint rh_WRJ2
